Commit message: add can interface

File: gf3_description/urdf/gf3_temp_arm_core.xacro (robot description, xacro)
@@ -1,8 +1,7 @@
 <?xml version="1.0" encoding="utf-8"?>
-<robot
-  name="gf3">
+<robot xmlns:xacro="http://www.ros.org/wiki/xacro"  name="robot">
   <link
     name="base_link">
-    <inertial>
+    <!-- <inertial>
       <origin
         xyz="0 0 0"
@@ -17,5 +16,5 @@
         iyz="0"
         izz="0" />
-    </inertial>
+    </inertial> -->
     <visual>
       <origin
@@ -44,5 +43,5 @@
   <link
     name="shoulder_1">
-    <inertial>
+    <!-- <inertial>
       <origin
         xyz="0.143483235103531 0.0250123355737991 0.702729587168112"
@@ -57,5 +56,5 @@
         iyz="9.38593559269322E-12"
         izz="0.000184029805378281" />
-    </inertial>
+    </inertial> -->
     <visual>
       <origin
