Commit message: URDF, joint update

File: gf3_description/urdf/gf3.xacro (robot description, xacro)
@@ -2,5 +2,11 @@
 <robot xmlns:xacro="http://www.ros.org/wiki/xacro"  name="robot">
     <xacro:arg name="prefix" default="" />
-    <xacro:include filename="gf3_temp_arm_core.xacro" />
+    <xacro:include filename="gf3.urdf" />
+    <link name="base_link"/>
+    <joint name="base_link-base_link_inertia" type="fixed">
+      <parent link="base_link" />
+      <child link="base_link_inertia" />
+      <origin xyz="0 0 0" rpy="0 0 0" />
+    </joint>
     <xacro:include filename="ros2_control.xacro" />
     <xacro:rrbot_ros2_control

File: gf3_description/urdf/ros2_control.xacro (robot description, xacro)
@@ -9,22 +9,36 @@
                 <param name="example_param_hw_slowdown">100</param>
             </hardware>
-            <joint name="shoulder_1_shoulder_2">
+            <joint name="shoulder_1-2">
                     <command_interface name="position">
-                        <param name="min">-1</param>
-                        <param name="max">1</param>
+                        <param name="min">-3.1416</param>
+                        <param name="max">3.1416</param>
                     </command_interface>
                     <state_interface name="position"/>
                 </joint>
-                <joint name="shoulder_2_shoulder_3">
+                <joint name="shoulder_2-3">
                     <command_interface name="position">
-                        <param name="min">-1</param>
-                        <param name="max">1</param>
+                        <param name="min">-0.5236</param>
+                        <param name="max">1.5708</param>
                     </command_interface>
                     <state_interface name="position"/>
                 </joint>
-                <joint name="shoulder_3_upper_arm">
+                <joint name="shoulder_3-upper">
                     <command_interface name="position">
-                        <param name="min">-1</param>
-                        <param name="max">1</param>
+                        <param name="min">-1.5708</param>
+                        <param name="max">1.5708</param>
+                    </command_interface>
+                    <state_interface name="position"/>
+                </joint>
+                <joint name="upper-elbow">
+                    <command_interface name="position">
+                        <param name="min">-1.5708</param>
+                        <param name="max">1.5708</param>
+                    </command_interface>
+                    <state_interface name="position"/>
+                </joint>
+                <joint name="elbow-lower">
+                    <command_interface name="position">
+                        <param name="min">-1.5708</param>
+                        <param name="max">1.5708</param>
                     </command_interface>
                     <state_interface name="position"/>
